Commit message: (ubr1_description) revert change in torso mass

File: ubr1_description/robots/ubr1_robot.urdf (robot description, URDF)
Before this commit: robot ubr1, 26 links, 25 joints
Links:
- link fixed_torso_link: mass 10.19400 -> 7.19400

Commit message: (ubr_controllers) add simulated gripper controller

File: ubr1_description/robots/ubr1_robot.urdf (robot description, URDF)
Before this commit: robot ubr1, 26 links, 25 joints
Joints:
- joint left_gripper_joint: limit lower=0.0 upper=0.045 effort=0.0 velocity=0.1 -> lower=0.0 upper=0.045 effort=28.0 velocity=0.1
- joint right_gripper_joint: limit lower=0.0 upper=0.045 effort=0.0 velocity=0.1 -> lower=0.0 upper=0.045 effort=28.0 velocity=0.1

Commit message: (ubr1_gazebo) torso lift working

File: ubr1_description/robots/ubr1_robot.urdf (robot description, URDF)
Before this commit: robot ubr1, 26 links, 25 joints
Joints:
- joint torso_lift_joint: limit lower=0.0 upper=0.3556 effort=37.802 velocity=0.05 -> lower=0.0 upper=0.3556 effort=450 velocity=0.05

Commit message: (ubr_controllers) add a simulated controller for the bellows joint

File: ubr1_description/robots/ubr1_robot.urdf (robot description, URDF)
Before this commit: robot ubr1, 26 links, 25 joints
Links:
- added link bellows_link, mass 0.1; visual mesh filename=package://ubr1_description/meshes/bellows_link.STL
Joints:
- added joint bellows_joint: type prismatic, parent torso_lift_link, child bellows_link, origin xyz=0.0047367 0 -0.1823 rpy=1.5708 -2.4652E-32 -1.5708, axis 0 1 0, limit lower=-0.1778 upper=0.0 effort=25.0 velocity=0.0

Commit message: (ubr1_description) remove collision meshes

File: ubr1_description/robots/ubr1_robot.urdf (robot description, URDF)
Before this commit: robot ubr1, 27 links, 26 joints
Links:
- link base_laser_link: geometry visual mesh filename=package://ubr1_description/meshes/base_laser_link.STL
- link base_link: geometry collision cylinder length=0.28 radius=0.25; visual mesh filename=package://ubr1_description/meshes/base_link.STL
- link elbow_flex_link: geometry visual mesh filename=package://ubr1_description/meshes/elbow_flex_link.STL
- link estop_link: geometry visual mesh filename=package://ubr1_description/meshes/estop_link.STL
- link fixed_bellows_link: geometry visual mesh filename=package://ubr1_description/meshes/bellows_link.STL
- link fixed_torso_link: geometry collision box size=0.20 0.40 0.32; visual mesh filename=package://ubr1_description/meshes/fixed_torso_link.STL
- link forearm_roll_link: geometry collision box size=0.275 0.15 0.10; visual mesh filename=package://ubr1_description/meshes/forearm_roll_link.STL
- link gripper_link: geometry collision box size=0.08 0.102 0.05; visual mesh filename=package://ubr1_description/meshes/gripper_link.STL
- link head_camera_link: geometry visual mesh filename=package://ubr1_description/meshes/head_camera_link.STL
- link head_pan_link: geometry collision box size=0.30 0.29 0.11; visual mesh filename=package://ubr1_description/meshes/head_pan_link.STL
- link head_tilt_link: geometry collision box size=0.10 0.29 0.10; visual mesh filename=package://ubr1_description/meshes/head_tilt_link.STL
- link left_gripper_finger_link: geometry collision box size=0.06 0.01 0.022; visual mesh filename=package://ubr1_description/meshes/left_gripper_finger_link.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
- link right_gripper_finger_link: geometry collision box size=0.06 0.01 0.022; visual mesh filename=package://ubr1_description/meshes/right_gripper_finger_link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
- link shoulder_lift_link: geometry collision cylinder length=0.23 radius=0.09; visual mesh filename=package://ubr1_description/meshes/shoulder_lift_link.STL
- link shoulder_pan_link: geometry collision cylinder length=0.19 radius=0.115; visual mesh filename=package://ubr1_description/meshes/shoulder_pan_link.STL
- link torso_lift_link: geometry collision box size=0.20 0.32 0.58; visual mesh filename=package://ubr1_description/meshes/torso_lift_link.STL
- link upperarm_roll_link: geometry collision cylinder length=0.255 radius=0.075; visual mesh filename=package://ubr1_description/meshes/upperarm_roll_link.STL
- link wrist_flex_link: geometry visual mesh filename=package://ubr1_description/meshes/wrist_flex_link.STL
- link wrist_roll_link: geometry visual mesh filename=package://ubr1_description/meshes/wrist_roll_link.STL
Joints:
- joint base_l_wheel_joint: origin xyz=0 0.17 0.05715 rpy=0 0 0 -> xyz=0 0.17 0.05615 rpy=0 0 0
- joint base_r_wheel_joint: origin xyz=0 -0.17 0.05715 rpy=0 0 0 -> xyz=0 -0.17 0.05615 rpy=0 0 0

File: ubr1_gazebo/robots/ubr1_robot.urdf.xacro (robot description, xacro)
@@ -72,5 +72,5 @@
     <sensor type="depth" name="camera">
       <always_on>true</always_on>
-      <update_rate>20.0</update_rate>
+      <update_rate>15.0</update_rate>
       <camera>
         <horizontal_fov>1.047197</horizontal_fov>

Commit message: (ubr1_gazebo) tune base damping and friction -- matches real robot effort/acceleration profile

File: ubr1_description/robots/ubr1_robot.urdf (robot description, URDF)
Before this commit: robot ubr1, 27 links, 26 joints
Joints:
- joint base_l_wheel_joint: limit effort=8.0 velocity=20.0 -> effort=12.0 velocity=20.0
- joint base_r_wheel_joint: limit effort=8.0 velocity=20.0 -> effort=12.0 velocity=20.0

File: ubr1_gazebo/robots/ubr1_robot.urdf.xacro (robot description, xacro)
@@ -5,6 +5,6 @@
     <kp>100000000.0</kp>
     <kd>10.0</kd>
-    <mu1>0</mu1>
-    <mu2>0</mu2>
+    <mu1>0.5</mu1>
+    <mu2>0.5</mu2>
     <fdir1>1 0 0</fdir1>
     <maxVel>10.0</maxVel>

Commit message: (ubr1_description) update meshes, urdf for full real time

File: ubr1_description/robots/ubr1_robot.urdf (robot description, URDF)
Before this commit: robot ubr1, 27 links, 26 joints
Links:
- removed link gripper_led_link
- added link base_inertia, mass 35.0237183
- link base_laser_link: geometry collision box size=0.01 0.01 0.01; visual mesh filename=package://ubr1_description/meshes/base_laser_link.STL
- link base_link: mass 35.0237183 -> None
- link bellows_link: geometry collision box size=0.01 0.01 0.01; visual mesh filename=package://ubr1_description/meshes/bellows_link.STL
- link elbow_flex_link: geometry collision cylinder length=0.05 radius=0.045; visual mesh filename=package://ubr1_description/meshes/elbow_flex_link.STL
- link estop_link: geometry collision box size=0.01 0.01 0.01; visual mesh filename=package://ubr1_description/meshes/estop_link.STL
- link fixed_bellows_link: geometry collision box size=0.01 0.01 0.01; visual mesh filename=package://ubr1_description/meshes/bellows_link.STL
- link forearm_roll_link: geometry collision mesh filename=package://ubr1_description/meshes/forearm_roll_link_col.STL; visual mesh filename=package://ubr1_description/meshes/forearm_roll_link.STL
- link gripper_link: mass 0.0548736502934717 -> 0.4218; geometry collision mesh filename=package://ubr1_description/meshes/gripper_link_col.STL; visual mesh filename=package://ubr1_description/meshes/gripper_link.STL
- link head_camera_link: geometry collision box size=0.01 0.01 0.01; visual mesh filename=package://ubr1_description/meshes/head_camera_link.STL
- link left_wheel_link: geometry collision cylinder length=0.03 radius=0.06; visual mesh filename=package://ubr1_description/meshes/left_wheel_link.STL
- link right_wheel_link: geometry collision cylinder length=0.03 radius=0.06; visual mesh filename=package://ubr1_description/meshes/right_wheel_link.STL
- link shoulder_lift_link: geometry collision mesh filename=package://ubr1_description/meshes/shoulder_lift_link_col.STL; visual mesh filename=package://ubr1_description/meshes/shoulder_lift_link.STL
- link shoulder_pan_link: geometry collision mesh filename=package://ubr1_description/meshes/shoulder_pan_link_col.STL; visual mesh filename=package://ubr1_description/meshes/shoulder_pan_link.STL
- link torso_lift_link: geometry collision mesh filename=package://ubr1_description/meshes/torso_lift_link_col.STL; visual mesh filename=package://ubr1_description/meshes/torso_lift_link.STL
- link upperarm_roll_link: geometry collision mesh filename=package://ubr1_description/meshes/upperarm_roll_link_col.STL; visual mesh filename=package://ubr1_description/meshes/upperarm_roll_link.STL
- link wrist_flex_link: geometry collision cylinder length=0.05 radius=0.04125; visual mesh filename=package://ubr1_description/meshes/wrist_flex_link.STL
- link wrist_roll_link: mass 0.4218 -> None; geometry collision cylinder length=0.05 radius=0.02; visual cylinder length=0.05 radius=0.02
Joints:
- removed joint gripper_led_joint
- added joint base_inertia_joint: type fixed, parent base_link, child base_inertia, origin xyz=0 0 0 rpy=0 0 0
- joint gripper_joint: origin xyz=0.110999999999998 0.0015000000000001 0 rpy=0 0 0 -> xyz=0 0 0 rpy=0 0 0
- joint left_gripper_joint: origin xyz=0 0 0 rpy=0 0 0 -> xyz=0.111 0 0 rpy=0 0 0
- joint right_gripper_joint: origin xyz=0 0 0 rpy=0 0 0 -> xyz=0.111 0 0 rpy=0 0 0
- joint shoulder_pan_joint: limit lower=-1.44862328 upper=1.44862328 effort=6.712 velocity=1.30899694 -> lower=-1.3962634 upper=1.3962634 effort=6.712 velocity=1.30899694

Commit message: (ubr1_gazebo) restore torso lift joint to working

File: ubr1_description/robots/ubr1_robot.urdf (robot description, URDF)
Before this commit: robot ubr1, 27 links, 26 joints
Joints:
- joint torso_lift_joint: limit lower=0.0 upper=0.3556 effort=450 velocity=0.05 -> lower=0.0 upper=0.3556 effort=450 velocity=0.1

Commit message: (ubr1_description) raise wheels, stops oscilliations in sim

File: ubr1_description/robots/ubr1_robot.urdf (robot description, URDF)
Before this commit: robot ubr1, 27 links, 26 joints
Joints:
- joint base_l_wheel_joint: origin xyz=0 0.17 0.05615 rpy=0 0 0 -> xyz=0 0.17 0.05735 rpy=0 0 0
- joint base_r_wheel_joint: origin xyz=0 -0.17 0.05615 rpy=0 0 0 -> xyz=0 -0.17 0.05735 rpy=0 0 0

Commit message: (ubr1_description) tweak wheel height again

File: ubr1_description/robots/ubr1_robot.urdf (robot description, URDF)
Before this commit: robot ubr1, 27 links, 26 joints
Joints:
- joint base_l_wheel_joint: origin xyz=0 0.17 0.05735 rpy=0 0 0 -> xyz=0 0.17 0.05725 rpy=0 0 0
- joint base_r_wheel_joint: origin xyz=0 -0.17 0.05735 rpy=0 0 0 -> xyz=0 -0.17 0.05725 rpy=0 0 0

Commit message: (ubr1_gazebo) update base collision mesh, base no longer moves around

File: ubr1_description/robots/ubr1_robot.urdf (robot description, URDF)
Before this commit: robot ubr1, 27 links, 26 joints
Links:
- link base_link: geometry collision mesh filename=package://ubr1_description/meshes/base_link_col.STL; visual mesh filename=package://ubr1_description/meshes/base_link.STL
Joints:
- joint base_l_wheel_joint: origin xyz=0 0.17 0.05725 rpy=0 0 0 -> xyz=0 0.17 0.05675 rpy=0 0 0
- joint base_r_wheel_joint: origin xyz=0 -0.17 0.05725 rpy=0 0 0 -> xyz=0 -0.17 0.05675 rpy=0 0 0

File: ubr1_gazebo/robots/ubr1_robot.urdf.xacro (robot description, xacro)
@@ -23,15 +23,13 @@
   <gazebo reference="right_gripper_finger_link">
     <material>Gazebo/Orange</material>
-    <mu1>1.0</mu1>
-    <mu2>1.0</mu2>
-    <minDepth>0.001</minDepth>
-    <maxVel>0.1</maxVel>
+    <mu1>10.0</mu1>
+    <mu2>10.0</mu2>
+    <fdir1>1 0 0</fdir1>
   </gazebo>
   <gazebo reference="left_gripper_finger_link">
     <material>Gazebo/Orange</material>
-    <mu1>1.0</mu1>
-    <mu2>1.0</mu2>
-    <minDepth>0.001</minDepth>
-    <maxVel>0.1</maxVel>
+    <mu1>10.0</mu1>
+    <mu2>10.0</mu2>
+    <fdir1>1 0 0</fdir1>
   </gazebo>
   <gazebo reference="torso_lift_link">
@@ -63,5 +61,5 @@
   </gazebo>
   <gazebo reference="right_wheel_link">
-    <kp>50000000.0</kp>
+    <kp>500000.0</kp>
     <kd>10.0</kd>
     <mu1>1.5</mu1>
@@ -73,5 +71,5 @@
   </gazebo>
   <gazebo reference="left_wheel_link">
-    <kp>50000000.0</kp>
+    <kp>500000.0</kp>
     <kd>10.0</kd>
     <mu1>1.5</mu1>
@@ -81,4 +79,10 @@
     <minDepth>0.003</minDepth>
     <material>Gazebo/Black</material>
+  </gazebo>
+  <gazebo reference="base_l_wheel_joint">
+    <implicitSpringDamper>1</implicitSpringDamper>
+  </gazebo>
+  <gazebo reference="base_r_wheel_joint">
+    <implicitSpringDamper>1</implicitSpringDamper>
   </gazebo>
   <!-- head camera -->

Commit message: expand range of gripper just a bit
was getting an out of range when gripper reports 0.0450000x due to noise

File: ubr1_description/robots/ubr1_robot.urdf (robot description, URDF)
Before this commit: robot ubr1, 27 links, 26 joints
Joints:
- joint left_gripper_joint: limit lower=0.0 upper=0.045 effort=28.0 velocity=0.1 -> lower=0.0 upper=0.046 effort=28.0 velocity=0.1
- joint right_gripper_joint: limit lower=0.0 upper=0.045 effort=28.0 velocity=0.1 -> lower=0.0 upper=0.046 effort=28.0 velocity=0.1

Commit message: revert urdf changes - fixed in drivers

File: ubr1_description/robots/ubr1_robot.urdf (robot description, URDF)
Before this commit: robot ubr1, 27 links, 26 joints
Joints:
- joint left_gripper_joint: limit lower=0.0 upper=0.046 effort=28.0 velocity=0.1 -> lower=0.0 upper=0.045 effort=28.0 velocity=0.1
